Commit message: 修改注释

File: urdf/coludata_arm.urdf (robot description, URDF)
Before this commit: robot coludata_arm, 8 links, 7 joints
Links:
- link base_link: geometry collision mesh filename=package://coludata_arm_ros/meshes/base_link.STL; visual mesh filename=package://coludata_arm_ros/meshes/base_link.STL
- link link1: geometry collision mesh filename=package://coludata_arm_ros/meshes/link1.STL; visual mesh filename=package://coludata_arm_ros/meshes/link1.STL
- link link2: geometry collision mesh filename=package://coludata_arm_ros/meshes/link2.STL; visual mesh filename=package://coludata_arm_ros/meshes/link2.STL
- link link3: geometry collision mesh filename=package://coludata_arm_ros/meshes/link3.STL; visual mesh filename=package://coludata_arm_ros/meshes/link3.STL
- link link4: geometry collision mesh filename=package://coludata_arm_ros/meshes/link4.STL; visual mesh filename=package://coludata_arm_ros/meshes/link4.STL
- link link5: geometry collision mesh filename=package://coludata_arm_ros/meshes/link5.STL; visual mesh filename=package://coludata_arm_ros/meshes/link5.STL
- link link6: geometry collision mesh filename=package://coludata_arm_ros/meshes/link6.STL; visual mesh filename=package://coludata_arm_ros/meshes/link6.STL
- link link7: geometry collision mesh filename=package://coludata_arm_ros/meshes/link7.STL; visual mesh filename=package://coludata_arm_ros/meshes/link7.STL
Joints:
- joint joint2: origin xyz=0 0 0 rpy=3.1416 -1.5708 1.5708 -> xyz=0 0 0 rpy=0.0 -1.5708 -1.5708
- joint joint3: origin xyz=0 0 0 rpy=1.5708 1.5708 0 -> xyz=0 0 0 rpy=1.5708 -1.5708 0
- joint joint4: origin xyz=0 0 0.3115 rpy=-1.5708 0 0 -> xyz=0 0 0.3115 rpy=1.5708 3.141592653589793 0
- joint joint5: origin xyz=0 0 0 rpy=1.5708 0 0 -> xyz=0 0 0 rpy=1.5708 3.141592653589793 0

Commit message: 更换了urdf和mesh文件

File: urdf/coludata_arm.urdf (robot description, URDF)
Before this commit: robot coludata_arm, 8 links, 7 joints
Links:
- link base_link: mass 2.1478 -> 0.96109
- link link1: mass 2.2321 -> 0.93379
- link link2: mass 0.29205 -> 0.6118
- link link3: mass 0.35003 -> 0.66978
- link link4: mass 0.15961 -> 0.50928
- link link5: mass 0.19653 -> 0.33845
- link link6: mass 0.10831 -> 0.25257
- link link7: mass 0.032625 -> 0.032648
Joints:
- joint joint1: axis 0 0 1 -> 0 0 -1; limit lower=-3.14159 upper=3.14159 effort=100 velocity=1.0 -> lower=-3.14 upper=3.14 effort=8 velocity=8; origin xyz=0 0 0.1196 rpy=0 0 0 -> xyz=0 0 0.1226 rpy=0 0 0
- joint joint2: axis 0 0 1 -> 0 0 -1; limit lower=-3.14159 upper=3.14159 effort=100 velocity=1.0 -> lower=-3.14 upper=3.14 effort=8 velocity=8; origin xyz=0 0 0 rpy=0.0 -1.5708 -1.5708 -> xyz=0 0 0 rpy=1.5708 -1.5708 0
- joint joint3: axis 0 0 1 -> 0 0 -1; limit lower=-3.14159 upper=3.14159 effort=100 velocity=1.0 -> lower=-3.14 upper=3.14 effort=8 velocity=8; origin xyz=0 0 0 rpy=1.5708 -1.5708 0 -> xyz=0 -0.3115 0 rpy=1.5708 1.5708 0
- joint joint4: axis 0 0 1 -> 0 0 -1; limit lower=-3.14159 upper=3.14159 effort=100 velocity=1.0 -> lower=-3.14 upper=3.14 effort=8 velocity=8; origin xyz=0 0 0.3115 rpy=1.5708 3.141592653589793 0 -> xyz=0 0 0 rpy=-1.5708 0 0
- joint joint5: axis 0 0 1 -> 0 0 -1; limit lower=-3.14159 upper=3.14159 effort=100 velocity=1.0 -> lower=-3.14 upper=3.14 effort=8 velocity=8; origin xyz=0 0 0 rpy=1.5708 3.141592653589793 0 -> xyz=0 -0.268 0 rpy=1.5708 0 0
- joint joint6: limit lower=-3.14159 upper=3.14159 effort=100 velocity=1.0 -> lower=-3.14 upper=3.14 effort=8 velocity=8; origin xyz=0 0 0.268 rpy=1.5708 -1.5708 0.0 -> xyz=0 0 0 rpy=1.5708 -1.5708 0
- joint joint7: limit lower=-3.14159 upper=3.14159 effort=100 velocity=1.0 -> lower=-3.14 upper=3.14 effort=8 velocity=8

Commit message: 增加了注释

File: urdf/coludata_arm.urdf (robot description, URDF)
Before this commit: robot coludata_arm, 8 links, 7 joints
Joints:
- joint joint2: origin xyz=0 0 0 rpy=1.5708 -1.5708 0 -> xyz=0 0 0 rpy=0.0 -1.5708 -1.5708
- joint joint6: origin xyz=0 0 0 rpy=1.5708 -1.5708 0 -> xyz=0 0 0 rpy=-1.5707926535897934 -1.5707926535897934 0
